File: src/hc_solder.kicad_pcb (KiCad board)
At the start: 2 copper layers, 60 x 50 mm, 9 parts, among them Q1 BC547

Commit message: Add files via upload
Parts:
- added G***: LOGO, LOGO, F.Cu at (130.0, 50.0)
Other:
- outline, holes or cut-outs redrawn
